File: Plus4Plus8.sch (KiCad schematic (older format))
At the start: 22 parts, among them CN1 JOY1, CN2 JOY2, CN3 JOY3, CN4 JOY4, CN5 JOY5, CN6 JOY6, CN7 JOY7, CN8 JOY8, CN9 PLUS4_USERPORT, U1 CD4051B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

Commit message: Initial layout
Parts:
- added C1, C2, C3, C4, C5: 100n, symbol Device:C
- added C6: 100u, symbol Device:CP1
Connections:
- net +5V: now also C1.1, C2.1, C3.1, C4.1, C5.1, C6.1
- net GND: now also C1.2, C2.2, C3.2, C4.2, C5.2, C6.2
Other:
- moved on the sheet: CN1, CN2, CN3, CN4, CN5, CN6, CN7, CN8, CN9, RN1, RN2, RN3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

Commit message: New layout, way funnier
Parts:
- removed CN9: PLUS4_USERPORT, Plus4Plus8:PLUS4_USERPORT, symbol PLUS4_USERPORT:PLUS4_USERPORT
- added CN9: DB15F, Connector_Dsub:DSUB-15_Female_EdgeMount_P2.77mm, symbol Connector:DB15_Female_MountingHoles
- CN1, CN2, CN3, CN4, CN5, CN6, CN7, CN8: footprint Plus4Plus8:DB_9M -> Connector_Dsub:DSUB-9_Male_EdgeMount_P2.77mm
- U1, U2, U3, U4, U5: footprint Package_DIP:DIP-16_W7.62mm_LongPads -> Package_DIP:DIP-16_W7.62mm_Socket_LongPads
Connections:
- net +5V: now also CN9.1, CN9.9 (P9)
- net GND: now also CN9.0 (PAD), CN9.15 (P15), CN9.8
- net d0: now also CN9.2
- net d1: now also CN9.3
- net d2: now also CN9.4
- net d3: now also CN9.5
- net d4: now also CN9.10 (P10)
- net d5: now also CN9.11 (P111)
- net d6: now also CN9.12 (P12)
- net d7: now also CN9.13 (P13)
- new net ~reset: CN9.6
- no-connect marks 19 -> 10
Changed lines of the file:
@@
 F 0 "U1" H 12920 3660 50  0000 C CNN
 F 1 "CD4051B" H 12860 2340 50  0000 C CNN
-F 2 "Package_DIP:DIP-16_W7.62mm_LongPads" H 12755 2255 50  0001 L CNN
+F 2 "Package_DIP:DIP-16_W7.62mm_Socket_LongPads" H 12755 2255 50  0001 L CNN
 F 3 "http://www.ti.com/lit/ds/symlink/cd4052b.pdf" H 12585 3105 50  0001 C CNN
 	1    12605 3005
@@
 $EndComp
 $Comp
-L PLUS4_USERPORT:PLUS4_USERPORT CN9
-U 1 1 63202686
-P 3145 2740
-F 0 "CN9" H 3145 3655 50  0000 C CNN
-F 1 "PLUS4_USERPORT" H 3145 3564 50  0000 C CNN
-F 2 "Plus4Plus8:PLUS4_USERPORT" H 3145 2740 50  0001 C CNN
-F 3 "DOCUMENTATION" H 3145 2740 50  0001 C CNN
-	1    3145 2740
-	1    0    0    -1
-$EndComp
-Wire Wire Line
-	3895 2190 4020 2190
-Wire Wire Line
-	4020 2190 4020 3290
-$Comp
-L power:GND #PWR0101
-U 1 1 63203F94
-P 4020 3440
-F 0 "#PWR0101" H 4020 3190 50  0001 C CNN
-F 1 "GND" H 4025 3267 50  0000 C CNN
-F 2 "" H 4020 3440 50  0001 C CNN
-F 3 "" H 4020 3440 50  0001 C CNN
-	1    4020 3440
-	1    0    0    -1
-$EndComp
-Wire Wire Line
-	3895 3290 4020 3290
-Connection ~ 4020 3290
-Wire Wire Line
-	4020 3290 4020 3440
-Wire Wire Line
-	2395 2190 2270 2190
-Wire Wire Line
-	2270 2190 2270 3290
-$Comp
 L power:GND #PWR0102
 U 1 1 632045C2
-P 2270 3440
-F 0 "#PWR0102" H 2270 3190 50  0001 C CNN
-F 1 "GND" H 2275 3267 50  0000 C CNN
-F 2 "" H 2270 3440 50  0001 C CNN
-F 3 "" H 2270 3440 50  0001 C CNN
-	1    2270 3440
-	-1   0    0    -1
-$EndComp
-Wire Wire Line
-	2395 3290 2270 3290
-Connection ~ 2270 3290
-Wire Wire Line
-	2270 3290 2270 3440
-NoConn ~ 2395 3190
-NoConn ~ 2395 3090
-NoConn ~ 2395 2990
-NoConn ~ 2395 2890
-NoConn ~ 3895 2390
-NoConn ~ 3895 2490
-NoConn ~ 3895 2590
-NoConn ~ 3895 2790
-NoConn ~ 3895 3090
-NoConn ~ 3895 3190
-NoConn ~ 2395 2390
-Wire Wire Line
-	2395 2290 2150 2290
+P 3245 4160
+F 0 "#PWR0102" H 3245 3910 50  0001 C CNN
+F 1 "GND" H 3250 3987 50  0000 C CNN
+F 2 "" H 3245 4160 50  0001 C CNN
+F 3 "" H 3245 4160 50  0001 C CNN
+	1    3245 4160
+	-1   0    0    -1
+$EndComp
 $Comp
 L power:+5V #PWR0103
 U 1 1 63206366
-P 2150 1760
-F 0 "#PWR0103" H 2150 1610 50  0001 C CNN
-F 1 "+5V" H 2165 1933 50  0000 C CNN
-F 2 "" H 2150 1760 50  0001 C CNN
-F 3 "" H 2150 1760 50  0001 C CNN
-	1    2150 1760
-	1    0    0    -1
-$EndComp
-Wire Wire Line
-	2395 2490 2150 2490
-Wire Wire Line
-	2395 2590 2150 2590
-Wire Wire Line
-	2395 2690 2150 2690
-Wire Wire Line
-	2395 2790 2150 2790
-Wire Wire Line
-	4140 2290 3895 2290
-Wire Wire Line
-	4140 2690 3895 2690
-Wire Wire Line
-	4140 2890 3895 2890
-Wire Wire Line
-	4140 2990 3895 2990
-Entry Wire Line
-	4140 2290 4240 2390
-Entry Wire Line
-	4140 2690 4240 2790
-Entry Wire Line
-	4140 2890 4240 2990
-Entry Wire Line
-	4140 2990 4240 3090
-Entry Wire Line
-	2050 2390 2150 2490
-Entry Wire Line
-	2050 2490 2150 2590
-Entry Wire Line
-	2050 2590 2150 2690
-Entry Wire Line
-	2050 2690 2150 2790
-Wire Bus Line
-	2050 3885 4240 3885
-Text Label 4140 2290 2    50   ~ 0
+P 3245 2120
+F 0 "#PWR0103" H 3245 1970 50  0001 C CNN
+F 1 "+5V" H 3260 2293 50  0000 C CNN
+F 2 "" H 3245 2120 50  0001 C CNN
+F 3 "" H 3245 2120 50  0001 C CNN
+	1    3245 2120
+	1    0    0    -1
+$EndComp
+Entry Wire Line
+	3315 2525 3415 2625
+Entry Wire Line
+	3315 3225 3415 3325
+Entry Wire Line
+	3315 3025 3415 3125
+Entry Wire Line
+	3315 2725 3415 2825
+Entry Wire Line
+	3415 3025 3315 2925
+Entry Wire Line
+	3415 3225 3315 3125
+Entry Wire Line
+	3415 2725 3315 2625
+Entry Wire Line
+	3415 2925 3315 2825
+Text Label 3315 2525 2    50   ~ 0
 d0
-Text Label 4140 2690 2    50   ~ 0
+Text Label 3315 3225 2    50   ~ 0
 d7
-Text Label 4140 2890 2    50   ~ 0
+Text Label 3315 3025 2    50   ~ 0
 d6
-Text Label 4140 2990 2    50   ~ 0
+Text Label 3315 2725 2    50   ~ 0
 d1
-Text Label 2150 2490 0    50   ~ 0
+Text Label 3315 2925 2    50   ~ 0
 d2
-Text Label 2150 2590 0    50   ~ 0
+Text Label 3315 3125 2    50   ~ 0
 d3
-Text Label 2150 2690 0    50   ~ 0
+Text Label 3315 2625 2    50   ~ 0
 d4
-Text Label 2150 2790 0    50   ~ 0
+Text Label 3315 2825 2    50   ~ 0
 d5
 $Comp
@@
 F 0 "CN1" H 5979 1777 50  0000 L CNN
 F 1 "JOY1" H 5979 1686 50  0000 L CNN
-F 2 "Plus4Plus8:DB_9M" H 5800 1775 50  0001 C CNN
+F 2 "Connector_Dsub:DSUB-9_Male_EdgeMount_P2.77mm" H 5800 1775 50  0001 C CNN
 F 3 " ~" H 5800 1775 50  0001 C CNN
 	1    5800 1775
@@
 F 0 "CN3" H 5718 7872 50  0000 C CNN
 F 1 "JOY3" H 5718 7781 50  0000 C CNN
-F 2 "Plus4Plus8:DB_9M" H 5800 7180 50  0001 C CNN
+F 2 "Connector_Dsub:DSUB-9_Male_EdgeMount_P2.77mm" H 5800 7180 50  0001 C CNN
 F 3 " ~" H 5800 7180 50  0001 C CNN
 	1    5800 7180
@@
 F 0 "CN4" H 5713 10722 50  0000 C CNN
 F 1 "JOY4" H 5713 10631 50  0000 C CNN
-F 2 "Plus4Plus8:DB_9M" H 5795 10030 50  0001 C CNN
+F 2 "Connector_Dsub:DSUB-9_Male_EdgeMount_P2.77mm" H 5795 10030 50  0001 C CNN
 F 3 " ~" H 5795 10030 50  0001 C CNN
 	1    5795 10030
@@
 F 0 "CN5" H 8938 2467 50  0000 C CNN
 F 1 "JOY5" H 8938 2376 50  0000 C CNN
-F 2 "Plus4Plus8:DB_9M" H 9020 1775 50  0001 C CNN
+F 2 "Connector_Dsub:DSUB-9_Male_EdgeMount_P2.77mm" H 9020 1775 50  0001 C CNN
 F 3 " ~" H 9020 1775 50  0001 C CNN
 	1    9020 1775
@@
 F 0 "CN6" H 8938 5107 50  0000 C CNN
 F 1 "JOY6" H 8938 5016 50  0000 C CNN
-F 2 "Plus4Plus8:DB_9M" H 9020 4415 50  0001 C CNN
+F 2 "Connector_Dsub:DSUB-9_Male_EdgeMount_P2.77mm" H 9020 4415 50  0001 C CNN
 F 3 " ~" H 9020 4415 50  0001 C CNN
 	1    9020 4415
@@
 F 0 "CN7" H 8938 7872 50  0000 C CNN
 F 1 "JOY7" H 8938 7781 50  0000 C CNN
-F 2 "Plus4Plus8:DB_9M" H 9020 7180 50  0001 C CNN
+F 2 "Connector_Dsub:DSUB-9_Male_EdgeMount_P2.77mm" H 9020 7180 50  0001 C CNN
 F 3 " ~" H 9020 7180 50  0001 C CNN
 	1    9020 7180
@@
 F 0 "CN8" H 8933 10722 50  0000 C CNN
 F 1 "JOY8" H 8933 10631 50  0000 C CNN
-F 2 "Plus4Plus8:DB_9M" H 9015 10030 50  0001 C CNN
+F 2 "Connector_Dsub:DSUB-9_Male_EdgeMount_P2.77mm" H 9015 10030 50  0001 C CNN
 F 3 " ~" H 9015 10030 50  0001 C CNN
 	1    9015 10030
@@
 F 0 "CN2" H 5718 5107 50  0000 C CNN
 F 1 "JOY2" H 5718 5016 50  0000 C CNN
-F 2 "Plus4Plus8:DB_9M" H 5800 4415 50  0001 C CNN
+F 2 "Connector_Dsub:DSUB-9_Male_EdgeMount_P2.77mm" H 5800 4415 50  0001 C CNN
 F 3 " ~" H 5800 4415 50  0001 C CNN
 	1    5800 4415
@@
 F 0 "U2" H 12920 6315 50  0000 C CNN
 F 1 "CD4051B" H 12860 4995 50  0000 C CNN
-F 2 "Package_DIP:DIP-16_W7.62mm_LongPads" H 12755 4910 50  0001 L CNN
+F 2 "Package_DIP:DIP-16_W7.62mm_Socket_LongPads" H 12755 4910 50  0001 L CNN
 F 3 "http://www.ti.com/lit/ds/symlink/cd4052b.pdf" H 12585 5760 50  0001 C CNN
 	1    12605 5660
@@
 F 0 "U3" H 12920 9065 50  0000 C CNN
 F 1 "CD4051B" H 12860 7745 50  0000 C CNN
-F 2 "Package_DIP:DIP-16_W7.62mm_LongPads" H 12755 7660 50  0001 L CNN
+F 2 "Package_DIP:DIP-16_W7.62mm_Socket_LongPads" H 12755 7660 50  0001 L CNN
 F 3 "http://www.ti.com/lit/ds/symlink/cd4052b.pdf" H 12585 8510 50  0001 C CNN
 	1    12605 8410
@@
 F 0 "U4" H 14845 4885 50  0000 C CNN
 F 1 "CD4051B" H 14785 3565 50  0000 C CNN
-F 2 "Package_DIP:DIP-16_W7.62mm_LongPads" H 14680 3480 50  0001 L CNN
+F 2 "Package_DIP:DIP-16_W7.62mm_Socket_LongPads" H 14680 3480 50  0001 L CNN
 F 3 "http://www.ti.com/lit/ds/symlink/cd4052b.pdf" H 14510 4330 50  0001 C CNN
 	1    14530 4230
@@
 F 0 "U5" H 14845 7615 50  0000 C CNN
 F 1 "CD4051B" H 14785 6295 50  0000 C CNN
-F 2 "Package_DIP:DIP-16_W7.62mm_LongPads" H 14680 6210 50  0001 L CNN
+F 2 "Package_DIP:DIP-16_W7.62mm_Socket_LongPads" H 14680 6210 50  0001 L CNN
 F 3 "http://www.ti.com/lit/ds/symlink/cd4052b.pdf" H 14510 7060 50  0001 C CNN
 	1    14530 6960
@@
 Wire Wire Line
 	10095 10330 11345 10330
-Wire Wire Line
-	2150 2290 2150 1760
-Text Label 4690 3885 2    50   ~ 0
-data_bus
-Wire Bus Line
-	4240 3885 4690 3885
-Connection ~ 4240 3885
 $Comp
 L power:+5V #PWR01
@@
 	1    0    0    -1
 $EndComp
+$Comp
+L Connector:DB15_Female_MountingHoles CN9
+U 1 1 636CDFF8
+P 2685 3025
+F 0 "CN9" H 2591 4017 50  0000 C CNN
+F 1 "DB15F" H 2591 3926 50  0000 C CNN
+F 2 "Connector_Dsub:DSUB-15_Female_EdgeMount_P2.77mm" H 2685 3025 50  0001 C CNN
+F 3 " ~" H 2685 3025 50  0001 C CNN
+	1    2685 3025
+	-1   0    0    -1
+$EndComp
+Wire Wire Line
+	2985 2325 3245 2325
+Wire Wire Line
+	3245 2120 3245 2325
+Wire Wire Line
+	2985 2425 3245 2425
+Wire Wire Line
+	3245 2425 3245 2325
+Connection ~ 3245 2325
+Wire Wire Line
+	2985 3625 3245 3625
+Wire Wire Line
+	3245 3625 3245 3725
+Wire Wire Line
+	2985 3725 3245 3725
+Connection ~ 3245 3725
+Wire Wire Line
+	3245 3725 3245 4050
+Wire Wire Line
+	2685 3925 2685 4050
+Wire Wire Line
+	2685 4050 3245 4050
+Connection ~ 3245 4050
+Wire Wire Line
+	3245 4050 3245 4160
+Wire Wire Line
+	2985 2525 3315 2525
+Wire Bus Line
+	3415 4050 3875 4050
+Text Label 3875 4050 2    50   ~ 0
+data_bus
+Wire Wire Line
+	2985 2625 3315 2625
+Wire Wire Line
+	2985 2725 3315 2725
+Wire Wire Line
+	2985 2825 3315 2825
+Wire Wire Line
+	2985 2925 3315 2925
+Wire Wire Line
+	2985 3025 3315 3025
+Wire Wire Line
+	2985 3125 3315 3125
+Wire Wire Line
+	2985 3225 3315 3225
+Wire Wire Line
+	2985 3325 3315 3325
+NoConn ~ 2985 3425
+NoConn ~ 2985 3525
 Wire Bus Line
 	13345 2405 13345 2805
@@
 	15270 6360 15270 6760
 Wire Bus Line
-	2050 2390 2050 3885
-Wire Bus Line
-	4240 2390 4240 3885
+	3415 2625 3415 4050
+Text Label 3315 3325 2    50   ~ 0
+~reset
 $EndSCHEMATC

Commit message: Routing in progress
Parts:
- C1, C2, C3, C4, C5: footprint (none) -> Capacitor_THT:C_Disc_D7.0mm_W2.5mm_P5.00mm
- C6: footprint (none) -> Capacitor_THT:CP_Radial_D6.3mm_P2.50mm
Connections:
- net at CN4.4, U4.12 (X3): now also RN4.3 (R2); no longer RN4.5 (R4)
- net at CN1.4, U4.13 (X0): now also RN1.3 (R2); no longer RN1.5 (R4)
- net at CN2.4, U4.14 (X1): now also RN2.3 (R2); no longer RN2.5 (R4)
- net at CN3.4, U4.15 (X2): now also RN3.3 (R2); no longer RN3.5 (R4)
- net at CN4.6, U5.12 (X3): now also RN4.2 (R1); no longer RN4.6 (R5)
- net at CN1.6, U5.13 (X0): now also RN1.2 (R1); no longer RN1.6 (R5)
- net at CN2.6, U5.14 (X1): now also RN2.2 (R1); no longer RN2.6 (R5)
- net at CN3.6, U5.15 (X2): now also RN3.2 (R1); no longer RN3.6 (R5)
- net at CN4.1, U1.12 (X3): now also RN4.6 (R5); no longer RN4.2 (R1)
- net at CN1.1, U1.13 (X0): now also RN1.6 (R5); no longer RN1.2 (R1)
- net at CN2.1, U1.14 (X1): now also RN2.6 (R5); no longer RN2.2 (R1)
- net at CN3.1, U1.15 (X2): now also RN3.6 (R5); no longer RN3.2 (R1)
- net at CN1.2, U2.13 (X0): now also RN1.5 (R4); no longer RN1.3 (R2)
- net at CN2.2, U2.14 (X1): now also RN2.5 (R4); no longer RN2.3 (R2)
- net at CN3.2, U2.15 (X2): now also RN3.5 (R4); no longer RN3.3 (R2)
- net at CN4.2, U2.12 (X3): now also RN4.5 (R4); no longer RN4.3 (R2)

Commit message: Rough routing done except power
Connections:
- net at CN5.4, U4.1 (X4): now also RN5.3 (R2); no longer RN5.5 (R4)
- net at CN7.4, U4.2 (X6): now also RN7.3 (R2); no longer RN7.5 (R4)
- net at CN8.4, U4.4 (X7): now also RN8.3 (R2); no longer RN8.5 (R4)
- net at CN6.4, U4.5 (X5): now also RN6.3 (R2); no longer RN6.5 (R4)
- net at CN5.6, U5.1 (X4): now also RN5.2 (R1); no longer RN5.6 (R5)
- net at CN7.6, U5.2 (X6): now also RN7.2 (R1); no longer RN7.6 (R5)
- net at CN8.6, U5.4 (X7): now also RN8.2 (R1); no longer RN8.6 (R5)
- net at CN6.6, U5.5 (X5): now also RN6.2 (R1); no longer RN6.6 (R5)
- net at CN5.1, U1.1 (X4): now also RN5.6 (R5); no longer RN5.2 (R1)
- net at CN7.1, U1.2 (X6): now also RN7.6 (R5); no longer RN7.2 (R1)
- net at CN8.1, U1.4 (X7): now also RN8.6 (R5); no longer RN8.2 (R1)
- net at CN6.1, U1.5 (X5): now also RN6.6 (R5); no longer RN6.2 (R1)
- net at CN5.2, U2.1 (X4): now also RN5.5 (R4); no longer RN5.3 (R2)
- net at CN6.2, U2.5 (X5): now also RN6.5 (R4); no longer RN6.3 (R2)
- net at CN7.2, U2.2 (X6): now also RN7.5 (R4); no longer RN7.3 (R2)
- net at CN8.2, U2.4 (X7): now also RN8.5 (R4); no longer RN8.3 (R2)
