File: Plus4Plus8.kicad_pcb (KiCad board)
At the start: 2 copper layers, 89.2 x 87.9 mm, 28 parts, among them CN1 JOY1, CN2 JOY2, CN3 JOY3, CN4 JOY4, CN5 JOY5, CN6 JOY6, CN7 JOY7, CN8 JOY8, CN9 DB15F, U1 CD4051B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

Commit message: Almost there
Routing:
- net GND: vias 12 -> 32
Changed lines of the file:
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@@
     (thickness 1.6)
     (drawings 9)
-    (tracks 772)
+    (tracks 792)
     (zones 0)
     (modules 28)
@@
   (title_block
     (title Plus4Plus8)
-    (date 2022-09-02)
+    (date 2022-09-04)
     (rev 1git)
     (company SukkoPera)
@@
   (via (at 169.164 131.826) (size 0.6) (drill 0.4) (layers F.Cu B.Cu) (net 1))
   (via (at 166.116 133.35) (size 0.6) (drill 0.4) (layers F.Cu B.Cu) (net 1))
+  (via (at 134.62 133.858) (size 0.6) (drill 0.4) (layers F.Cu B.Cu) (net 1))
+  (via (at 133.731 131.826) (size 0.6) (drill 0.4) (layers F.Cu B.Cu) (net 1))
+  (via (at 136.779 133.35) (size 0.6) (drill 0.4) (layers F.Cu B.Cu) (net 1))
+  (via (at 115.824 115.697) (size 0.6) (drill 0.4) (layers F.Cu B.Cu) (net 1))
+  (via (at 114.3 112.649) (size 0.6) (drill 0.4) (layers F.Cu B.Cu) (net 1))
+  (via (at 113.792 114.808) (size 0.6) (drill 0.4) (layers F.Cu B.Cu) (net 1))
+  (via (at 189.103 114.808) (size 0.6) (drill 0.4) (layers F.Cu B.Cu) (net 1))
+  (via (at 188.595 112.649) (size 0.6) (drill 0.4) (layers F.Cu B.Cu) (net 1))
+  (via (at 187.071 115.697) (size 0.6) (drill 0.4) (layers F.Cu B.Cu) (net 1))
+  (via (at 108.585 85.344) (size 0.6) (drill 0.4) (layers F.Cu B.Cu) (net 1))
+  (via (at 109.474 87.376) (size 0.6) (drill 0.4) (layers F.Cu B.Cu) (net 1))
+  (via (at 109.982 83.693) (size 0.6) (drill 0.4) (layers F.Cu B.Cu) (net 1))
+  (via (at 194.31 85.344) (size 0.6) (drill 0.4) (layers F.Cu B.Cu) (net 1))
+  (via (at 193.421 87.376) (size 0.6) (drill 0.4) (layers F.Cu B.Cu) (net 1))
+  (via (at 192.913 83.693) (size 0.6) (drill 0.4) (layers F.Cu B.Cu) (net 1))
+  (via (at 150.114 103.759) (size 0.6) (drill 0.4) (layers F.Cu B.Cu) (net 1))
+  (via (at 152.019 103.759) (size 0.6) (drill 0.4) (layers F.Cu B.Cu) (net 1))
+  (via (at 152.019 105.537) (size 0.6) (drill 0.4) (layers F.Cu B.Cu) (net 1))
+  (via (at 150.114 105.537) (size 0.6) (drill 0.4) (layers F.Cu B.Cu) (net 1))
+  (via (at 152.019 107.315) (size 0.6) (drill 0.4) (layers F.Cu B.Cu) (net 1))
   (segment (start 152.694 94.090469) (end 151.374 95.410469) (width 0.5) (layer F.Cu) (net 2) (status 20))
   (segment (start 155.184 94.090469) (end 152.694 94.090469) (width 0.5) (layer F.Cu) (net 2) (status 10))
@@
   (via (at 146.304 130.048) (size 0.6) (drill 0.4) (layers F.Cu B.Cu) (net 43))
   (segment (start 151.638 130.048) (end 146.304 130.048) (width 0.25) (layer F.Cu) (net 43))
-  (segment (start 140.97 124.714) (end 146.304 130.048) (width 0.25) (layer B.Cu) (net 43))
   (segment (start 152.769 133.477) (end 152.769 131.179) (width 0.25) (layer F.Cu) (net 43) (status 10))
   (segment (start 152.769 131.179) (end 151.638 130.048) (width 0.25) (layer F.Cu) (net 43))
-  (segment (start 134.864 108.067) (end 140.97 114.173) (width 0.25) (layer B.Cu) (net 43))
-  (segment (start 134.864 101.710469) (end 134.864 108.067) (width 0.25) (layer B.Cu) (net 43) (status 10))
-  (segment (start 140.97 114.173) (end 140.97 124.714) (width 0.25) (layer B.Cu) (net 43))
+  (segment (start 140.97 124.714) (end 146.304 130.048) (width 0.25) (layer B.Cu) (net 43))
+  (segment (start 140.97 110.109) (end 140.97 124.714) (width 0.25) (layer B.Cu) (net 43))
+  (segment (start 134.864 104.003) (end 140.97 110.109) (width 0.25) (layer B.Cu) (net 43))
+  (segment (start 134.864 101.710469) (end 134.864 104.003) (width 0.25) (layer B.Cu) (net 43))
   (segment (start 157.1625 130.048) (end 153.035 130.048) (width 0.25) (layer F.Cu) (net 44))
   (segment (start 147.065996 129.286) (end 146.303996 128.524) (width 0.25) (layer F.Cu) (net 44))
@@
       )
     )
+  )
+  (zone (net 0) (net_name "") (layer B.Cu) (hatch edge 0.508)
+    (connect_pads (clearance 0.508))
+    (min_thickness 0.254)
+    (keepout (tracks allowed) (vias allowed) (copperpour not_allowed))
+    (fill (arc_segments 32) (thermal_gap 0.508) (thermal_bridge_width 0.508))
+    (polygon
+      (pts
+        (xy 148.7805 82.1055) (xy 146.1135 82.1055) (xy 146.1135 84.328) (xy 141.478 84.328) (xy 141.478 80.518)
+        (xy 148.7805 80.518)
+      )
+    )
+  )
+  (zone (net 0) (net_name "") (layer B.Cu) (hatch edge 0.508)
+    (connect_pads (clearance 0.508))
+    (min_thickness 0.254)
+    (keepout (tracks allowed) (vias allowed) (copperpour not_allowed))
+    (fill (arc_segments 32) (thermal_gap 0.508) (thermal_bridge_width 0.508))
+    (polygon
+      (pts
+        (xy 148.844 103.505) (xy 141.224 103.505) (xy 141.224 100.203) (xy 148.844 100.203)
+      )
+    )
+  )
+  (zone (net 0) (net_name "") (layer B.Cu) (hatch edge 0.508)
+    (connect_pads (clearance 0.508))
+    (min_thickness 0.254)
+    (keepout (tracks allowed) (vias allowed) (copperpour not_allowed))
+    (fill (arc_segments 32) (thermal_gap 0.508) (thermal_bridge_width 0.508))
+    (polygon
+      (pts
+        (xy 171.704 101.346) (xy 165.354 101.346) (xy 165.354 98.933) (xy 171.704 98.933)
+      )
+    )
+  )
+  (zone (net 0) (net_name "") (layer B.Cu) (hatch edge 0.508)
+    (connect_pads (clearance 0.508))
+    (min_thickness 0.254)
+    (keepout (tracks allowed) (vias allowed) (copperpour not_allowed))
+    (fill (arc_segments 32) (thermal_gap 0.508) (thermal_bridge_width 0.508))
+    (polygon
+      (pts
+        (xy 171.704 84.582) (xy 166.624 84.582) (xy 166.624 80.518) (xy 171.704 80.518)
+      )
+    )
