File: Plus4Plus8.kicad_pcb (KiCad board)
At the start: 2 copper layers, 89.2 x 87.9 mm, 28 parts, among them CN1 JOY1, CN2 JOY2, CN3 JOY3, CN4 JOY4, CN5 JOY5, CN6 JOY6, CN7 JOY7, CN8 JOY8, CN9 DB15F, U1 CD4051B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

Commit message: Ja ja ja
Routing:
- net Net-(CN3-Pad3): track 34.2 -> 39.8 mm
- net Net-(CN8-Pad1): track 78.5 -> 73.8 mm
- net Net-(CN1-Pad2): track 84.0 -> 86.5 mm
- net Net-(CN8-Pad2): track 59.2 -> 57.0 mm
- net Net-(CN1-Pad4): track 60.4 -> 62.0 mm
- net Net-(CN8-Pad6): track 40.4 -> 41.8 mm, vias 0 -> 1
- net Net-(CN5-Pad3): track 79.1 -> 77.9 mm
- net /d2: track 42.3 -> 43.4 mm
- net /d5: track 135.0 -> 136.0 mm
- net Net-(CN8-Pad4): track 35.6 -> 36.5 mm
- net Net-(CN3-Pad2): track 46.6 -> 45.9 mm
- net Net-(CN6-Pad6): track 81.0 -> 81.6 mm, vias 2 -> 3
- net GND: vias 32 -> 36
