File: WheelOfJoy.kicad_pcb (KiCad board)
At the start: 2 copper layers, 89.2 x 87.9 mm, 28 parts, among them CN1 JOY1, CN2 JOY2, CN3 JOY3, CN4 JOY4, CN5 JOY5, CN6 JOY6, CN7 JOY7, CN8 JOY8, CN9 DB15F, U1 CD4051B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

Commit message: Ready for V1 RC1
Parts:
- added V0: LOGO, WheelOfJoy:logo, F.Cu at (151.9, 67.6)
- added V1: OSHW_LOGO, WheelOfJoy:cc_by_nc_sa, F.Cu at (169.7, 107.0)
- added V2: PORT1_NO, WheelOfJoy:port1, F.Cu at (119.3, 116.6)
- added V3: PORT2_NO, WheelOfJoy:port2, F.Cu at (111.4, 89.7)
- added V4: PORT3_NO, WheelOfJoy:port3, F.Cu at (122.9, 64.3)
- added V5: PORT4_NO, WheelOfJoy:port4, F.Cu at (146.9, 52.7)
- added V6: PORT5_NO, WheelOfJoy:port5, F.Cu at (174.9, 59.8)
- added V7: PORT6_NO, WheelOfJoy:port6, F.Cu at (190.2, 82.3)
- added V8: PORT7_NO, WheelOfJoy:port7, F.Cu at (190.0, 109.6)
- added V9: PORT8_NO, WheelOfJoy:port8, F.Cu at (171.6, 129.8)
Routing:
- net Net-(CN4-Pad6): track 86.4 -> 74.7 mm
- net Net-(CN4-Pad1): track 32.8 -> 28.8 mm
- net +5V: track 474.5 -> 471.3 mm, vias 9 -> 8
- net Net-(CN4-Pad2): track 39.0 -> 41.0 mm
- net Net-(CN3-Pad2): track 45.9 -> 47.7 mm
- net Net-(CN5-Pad3): track 77.9 -> 79.0 mm
- net /d5: track 136.0 -> 134.9 mm
Other:
- board text added: "+5V"
- board text added: "CC-BY-NC-SA SukkoPera 2022 github.com/SukkoPera/WheelOfJoy"
- board text added: "GND"
- board text added: "P0"
- board text added: "P1"
- board text added: "P2"
- board text added: "P3"
- board text added: "P4"
- board text added: "P5"
- board text added: "P6"
- board text added: "P7"

Commit message: Add series resistor on D1-D5
Parts:
- added RN9: 100, Resistor_THT:R_Array_SIP10, F.Cu at (162.8, 126.6)
- moved C6 7.58 mm to (167.4, 131.2), turned to 180 degrees
- moved V9 0.25 mm to (171.8, 129.8)
Connections:
- CN9 pad 10: /d4 -> Net-(CN9-Pad10)
- CN9 pad 2: /d0 -> Net-(CN9-Pad2)
- CN9 pad 3: /d1 -> Net-(CN9-Pad3)
- CN9 pad 4: /d2 -> Net-(CN9-Pad4)
- CN9 pad 5: /d3 -> Net-(CN9-Pad5)
Routing:
- net Net-(CN9-Pad2): track 0.00 -> 17.5 mm, vias 0 -> 3
- net /d0: track 75.4 -> 58.2 mm, vias 3 -> 2
- net Net-(CN9-Pad5): track 0.00 -> 17.1 mm
- net Net-(CN9-Pad4): track 0.00 -> 15.9 mm, vias 0 -> 2
- net /d2: track 43.4 -> 27.9 mm, vias 1 -> 0
- net /d3: track 40.1 -> 26.0 mm, vias 3 -> 0
- net Net-(CN9-Pad10): track 0.00 -> 10.0 mm, vias 0 -> 1
- net /d4: track 21.4 -> 11.9 mm, vias 2 -> 1
- net +5V: track 471.3 -> 461.8 mm, vias 8 -> 6
- net Net-(CN9-Pad3): track 0.00 -> 8.56 mm, vias 0 -> 2
- net /d1: track 53.2 -> 46.3 mm, vias 1 -> 0
- net GND: vias 36 -> 38

Commit message: Fix port labels And learn to count from 0 next time...
Parts:
- moved V8 1.97 mm to (188.0, 109.7)
- moved V6 0.94 mm to (174.2, 59.1)
- moved V5 0.91 mm to (147.8, 52.5)
- moved V7 0.52 mm to (189.7, 82.2)
- moved V4 0.23 mm to (122.7, 64.4)
Other:
- board text added: "V2"
