File: WheelOfJoy.sch (KiCad schematic (older format))
At the start: 28 parts, among them CN1 JOY1, CN2 JOY2, CN3 JOY3, CN4 JOY4, CN5 JOY5, CN6 JOY6, CN7 JOY7, CN8 JOY8, CN9 DB15F, U1 CD4051B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

Commit message: Ready for V1 RC1
Parts:
- added V0: LOGO, WheelOfJoy:logo, symbol void:Void
- added V1: OSHW_LOGO, WheelOfJoy:cc_by_nc_sa, symbol void:Void
- added V2: PORT1_NO, WheelOfJoy:port1, symbol void:Void
- added V3: PORT2_NO, WheelOfJoy:port2, symbol void:Void
- added V4: PORT3_NO, WheelOfJoy:port3, symbol void:Void
- added V5: PORT4_NO, WheelOfJoy:port4, symbol void:Void
- added V6: PORT5_NO, WheelOfJoy:port5, symbol void:Void
- added V7: PORT6_NO, WheelOfJoy:port6, symbol void:Void
- added V8: PORT7_NO, WheelOfJoy:port7, symbol void:Void
- added V9: PORT8_NO, WheelOfJoy:port8, symbol void:Void
Connections:
- no-connect marks 10 -> 11
Changed lines of the file:
@@
 Sheet 1 1
 Title "WheelOfJoy"
-Date "2022-09-03"
+Date "2022-09-04"
 Rev "1git"
 Comp "SukkoPera"
@@
 Wire Wire Line
 	9695 9695 9695 10330
+Connection ~ 9695 10330
+Wire Wire Line
+	9695 10330 11345 10330
+$Comp
+L void:Void V0
+U 1 1 631792FB
+P 14825 9580
+F 0 "V0" H 14903 9626 50  0000 L CNN
+F 1 "LOGO" H 14903 9535 50  0000 L CNN
+F 2 "WheelOfJoy:logo" H 14825 9580 50  0001 C CNN
+F 3 "" H 14825 9580 50  0001 C CNN
+	1    14825 9580
+	1    0    0    -1
+$EndComp
+$Comp
+L void:Void V1
+U 1 1 63197B4D
+P 14825 9770
+F 0 "V1" H 14903 9816 50  0000 L CNN
+F 1 "OSHW_LOGO" H 14903 9725 50  0000 L CNN
+F 2 "WheelOfJoy:cc_by_nc_sa" H 14825 9770 50  0001 C CNN
+F 3 "" H 14825 9770 50  0001 C CNN
+	1    14825 9770
+	1    0    0    -1
+$EndComp
+$Comp
+L void:Void V9
+U 1 1 6321012F
+P 15510 9770
+F 0 "V9" H 15588 9816 50  0000 L CNN
+F 1 "PORT8_NO" H 15588 9725 50  0000 L CNN
+F 2 "WheelOfJoy:port8" H 15510 9770 50  0001 C CNN
+F 3 "" H 15510 9770 50  0001 C CNN
+	1    15510 9770
+	1    0    0    -1
+$EndComp
+$Comp
+L void:Void V8
+U 1 1 632105FD
+P 15510 9565
+F 0 "V8" H 15588 9611 50  0000 L CNN
+F 1 "PORT7_NO" H 15588 9520 50  0000 L CNN
+F 2 "WheelOfJoy:port7" H 15510 9565 50  0001 C CNN
+F 3 "" H 15510 9565 50  0001 C CNN
+	1    15510 9565
+	1    0    0    -1
+$EndComp
+$Comp
+L void:Void V7
+U 1 1 632111D8
+P 15510 9360
+F 0 "V7" H 15588 9406 50  0000 L CNN
+F 1 "PORT6_NO" H 15588 9315 50  0000 L CNN
+F 2 "WheelOfJoy:port6" H 15510 9360 50  0001 C CNN
+F 3 "" H 15510 9360 50  0001 C CNN
+	1    15510 9360
+	1    0    0    -1
+$EndComp
+$Comp
+L void:Void V6
+U 1 1 63211B68
+P 15510 9155
+F 0 "V6" H 15588 9201 50  0000 L CNN
+F 1 "PORT5_NO" H 15588 9110 50  0000 L CNN
+F 2 "WheelOfJoy:port5" H 15510 9155 50  0001 C CNN
+F 3 "" H 15510 9155 50  0001 C CNN
+	1    15510 9155
+	1    0    0    -1
+$EndComp
+$Comp
+L void:Void V5
+U 1 1 63242F92
+P 15510 8950
+F 0 "V5" H 15588 8996 50  0000 L CNN
+F 1 "PORT4_NO" H 15588 8905 50  0000 L CNN
+F 2 "WheelOfJoy:port4" H 15510 8950 50  0001 C CNN
+F 3 "" H 15510 8950 50  0001 C CNN
+	1    15510 8950
+	1    0    0    -1
+$EndComp
+$Comp
+L void:Void V4
+U 1 1 6324393E
+P 15510 8745
+F 0 "V4" H 15588 8791 50  0000 L CNN
+F 1 "PORT3_NO" H 15588 8700 50  0000 L CNN
+F 2 "WheelOfJoy:port3" H 15510 8745 50  0001 C CNN
+F 3 "" H 15510 8745 50  0001 C CNN
+	1    15510 8745
+	1    0    0    -1
+$EndComp
+$Comp
+L void:Void V3
+U 1 1 63243948
+P 15510 8540
+F 0 "V3" H 15588 8586 50  0000 L CNN
+F 1 "PORT2_NO" H 15588 8495 50  0000 L CNN
+F 2 "WheelOfJoy:port2" H 15510 8540 50  0001 C CNN
+F 3 "" H 15510 8540 50  0001 C CNN
+	1    15510 8540
+	1    0    0    -1
+$EndComp
+$Comp
+L void:Void V2
+U 1 1 63243952
+P 15510 8335
+F 0 "V2" H 15588 8381 50  0000 L CNN
+F 1 "PORT1_NO" H 15588 8290 50  0000 L CNN
+F 2 "WheelOfJoy:port1" H 15510 8335 50  0001 C CNN
+F 3 "" H 15510 8335 50  0001 C CNN
+	1    15510 8335
+	1    0    0    -1
+$EndComp
+NoConn ~ 3315 3325
+$Comp
+L power:PWR_FLAG #FLG0101
+U 1 1 6331186A
+P 3380 2325
+F 0 "#FLG0101" H 3380 2400 50  0001 C CNN
+F 1 "PWR_FLAG" V 3380 2453 50  0000 L CNN
+F 2 "" H 3380 2325 50  0001 C CNN
+F 3 "~" H 3380 2325 50  0001 C CNN
+	1    3380 2325
+	0    1    1    0
+$EndComp
+Wire Wire Line
+	3245 2325 3380 2325
+$Comp
+L power:PWR_FLAG #FLG0102
+U 1 1 633433C0
+P 3470 3725
+F 0 "#FLG0102" H 3470 3800 50  0001 C CNN
+F 1 "PWR_FLAG" V 3470 3853 50  0000 L CNN
+F 2 "" H 3470 3725 50  0001 C CNN
+F 3 "~" H 3470 3725 50  0001 C CNN
+	1    3470 3725
+	0    1    1    0
+$EndComp
+Wire Wire Line
+	3245 3725 3470 3725
 Wire Bus Line
 	13345 2405 13345 2805
@@
 Wire Bus Line
 	3415 2625 3415 4050
-Connection ~ 9695 10330
-Wire Wire Line
-	9695 10330 11345 10330
 $EndSCHEMATC

Commit message: Add series resistor on D1-D5
Parts:
- added RN9: 100, Resistor_THT:R_Array_SIP10, symbol Device:R_Pack05_SIP_Split
Connections:
- net d0: now also RN9.8 (R4.2); no longer CN9.2
- net d1: now also RN9.4 (R2.2); no longer CN9.3
- net d2: now also RN9.10 (R5.2); no longer CN9.4
- net d3: now also RN9.2 (R1.2); no longer CN9.5
- net d4: now also RN9.6 (R3.2); no longer CN9.10 (P10)
- new net: CN9.10 (P10), RN9.5 (R3.1)
- new net: CN9.2, RN9.7 (R4.1)
- new net: CN9.3, RN9.3 (R2.1)
- new net: CN9.4, RN9.9 (R5.1)
- new net: CN9.5, RN9.1 (R1.1)
Other:
- moved on the sheet: CN9
Changed lines of the file:
@@
 Sheet 1 1
 Title "WheelOfJoy"
-Date "2022-09-04"
+Date "2022-09-12"
 Rev "1git"
 Comp "SukkoPera"
@@
 L Connector:DB15_Female_MountingHoles CN9
 U 1 1 636CDFF8
-P 2685 3025
-F 0 "CN9" H 2591 4017 50  0000 C CNN
-F 1 "DB15F" H 2591 3926 50  0000 C CNN
-F 2 "Connector_Dsub:DSUB-15_Female_EdgeMount_P2.77mm" H 2685 3025 50  0001 C CNN
-F 3 " ~" H 2685 3025 50  0001 C CNN
-	1    2685 3025
-	-1   0    0    -1
-$EndComp
-Wire Wire Line
-	2985 2325 3245 2325
+P 1915 3025
+F 0 "CN9" H 1821 4017 50  0000 C CNN
+F 1 "DB15F" H 1821 3926 50  0000 C CNN
+F 2 "Connector_Dsub:DSUB-15_Female_EdgeMount_P2.77mm" H 1915 3025 50  0001 C CNN
+F 3 " ~" H 1915 3025 50  0001 C CNN
+	1    1915 3025
+	-1   0    0    -1
+$EndComp
 Wire Wire Line
 	3245 2120 3245 2325
 Wire Wire Line
-	2985 2425 3245 2425
+	2215 2425 3245 2425
 Wire Wire Line
 	3245 2425 3245 2325
 Connection ~ 3245 2325
 Wire Wire Line
-	2985 3625 3245 3625
+	2215 3625 3245 3625
 Wire Wire Line
 	3245 3625 3245 3725
 Wire Wire Line
-	2985 3725 3245 3725
+	2215 3725 3245 3725
 Connection ~ 3245 3725
 Wire Wire Line
 	3245 3725 3245 4050
 Wire Wire Line
-	2685 3925 2685 4050
-Wire Wire Line
-	2685 4050 3245 4050
+	1915 3925 1915 4050
+Wire Wire Line
+	1915 4050 3245 4050
 Connection ~ 3245 4050
 Wire Wire Line
 	3245 4050 3245 4160
 Wire Wire Line
-	2985 2525 3315 2525
+	2215 2525 2490 2525
 Wire Bus Line
 	3415 4050 3875 4050
@@
 data_bus
 Wire Wire Line
-	2985 2625 3315 2625
-Wire Wire Line
-	2985 2725 3315 2725
-Wire Wire Line
-	2985 2825 3315 2825
-Wire Wire Line
-	2985 2925 3315 2925
-Wire Wire Line
-	2985 3025 3315 3025
-Wire Wire Line
-	2985 3125 3315 3125
-Wire Wire Line
-	2985 3225 3315 3225
-Wire Wire Line
-	2985 3325 3315 3325
-NoConn ~ 2985 3425
-NoConn ~ 2985 3525
+	2215 2625 2490 2625
+Wire Wire Line
+	2215 2725 2490 2725
+Wire Wire Line
+	2215 2825 3315 2825
+Wire Wire Line
+	2215 2925 2490 2925
+Wire Wire Line
+	2215 3025 3315 3025
+Wire Wire Line
+	2215 3125 2490 3125
+Wire Wire Line
+	2215 3225 3315 3225
+Wire Wire Line
+	2215 3325 3315 3325
+NoConn ~ 2215 3425
+NoConn ~ 2215 3525
 Text Label 3315 3325 2    50   ~ 0
 ~reset
@@
 Wire Wire Line
 	3245 3725 3470 3725
+$Comp
+L Device:R_Pack05_SIP_Split RN9
+U 2 1 63C155F9
+P 2640 2725
+F 0 "RN9" V 2600 2980 50  0000 C CNN
+F 1 "100" V 2524 2725 50  0001 C CNN
+F 2 "Resistor_THT:R_Array_SIP10" V 2560 2725 50  0001 C CNN
+F 3 "http://www.vishay.com/docs/31509/csc.pdf" H 2640 2725 50  0001 C CNN
+	2    2640 2725
+	0    1    1    0
+$EndComp
+$Comp
+L Device:R_Pack05_SIP_Split RN9
+U 3 1 63C16C68
+P 2640 2625
+F 0 "RN9" V 2600 2880 50  0000 C CNN
+F 1 "100" V 2524 2625 50  0001 C CNN
+F 2 "Resistor_THT:R_Array_SIP10" V 2560 2625 50  0001 C CNN
+F 3 "http://www.vishay.com/docs/31509/csc.pdf" H 2640 2625 50  0001 C CNN
+	3    2640 2625
+	0    1    1    0
+$EndComp
+$Comp
+L Device:R_Pack05_SIP_Split RN9
+U 4 1 63C17F96
+P 2640 2525
+F 0 "RN9" V 2600 2780 50  0000 C CNN
+F 1 "100" V 2524 2525 50  0001 C CNN
+F 2 "Resistor_THT:R_Array_SIP10" V 2560 2525 50  0001 C CNN
+F 3 "http://www.vishay.com/docs/31509/csc.pdf" H 2640 2525 50  0001 C CNN
+	4    2640 2525
+	0    1    1    0
+$EndComp
+$Comp
+L Device:R_Pack05_SIP_Split RN9
+U 5 1 63C19092
+P 2640 2925
+F 0 "RN9" V 2600 3175 50  0000 C CNN
+F 1 "100" V 2524 2925 50  0001 C CNN
+F 2 "Resistor_THT:R_Array_SIP10" V 2560 2925 50  0001 C CNN
+F 3 "http://www.vishay.com/docs/31509/csc.pdf" H 2640 2925 50  0001 C CNN
+	5    2640 2925
+	0    1    1    0
+$EndComp
+Wire Wire Line
+	2215 2325 3245 2325
+Wire Wire Line
+	2790 2525 3315 2525
+Wire Wire Line
+	2790 2725 3315 2725
+Wire Wire Line
+	2790 2925 3315 2925
+Wire Wire Line
+	2790 3125 3315 3125
+Wire Wire Line
+	2790 2625 3315 2625
 Wire Bus Line
 	13345 2405 13345 2805
@@
 Wire Bus Line
 	3415 2625 3415 4050
+$Comp
+L Device:R_Pack05_SIP_Split RN9
+U 1 1 63C134E3
+P 2640 3125
+F 0 "RN9" V 2600 3375 50  0000 C CNN
+F 1 "100" V 2600 2930 50  0000 C CNN
+F 2 "Resistor_THT:R_Array_SIP10" V 2560 3125 50  0001 C CNN
+F 3 "http://www.vishay.com/docs/31509/csc.pdf" H 2640 3125 50  0001 C CNN
+	1    2640 3125
+	0    1    1    0
+$EndComp
 $EndSCHEMATC

Commit message: Add notes on resistor arrays
Parts:
- RN1, RN2, RN3, RN4, RN5, RN6, RN7, RN8: Notes (none) -> Bussed
- RN9: Notes (none) -> Independent
Changed lines of the file:
@@
 Sheet 1 1
 Title "WheelOfJoy"
-Date "2022-09-12"
+Date "2022-11-06"
 Rev "1git"
 Comp "SukkoPera"
@@
 F 2 "Resistor_THT:R_Array_SIP6" V 7055 3880 50  0001 C CNN
 F 3 "http://www.vishay.com/docs/31509/csc.pdf" H 6680 3880 50  0001 C CNN
+F 4 "Bussed" H 6680 3880 50  0001 C CNN "Notes"
 	1    6680 3880
 	1    0    0    -1
@@
 F 2 "Resistor_THT:R_Array_SIP6" V 7055 6645 50  0001 C CNN
 F 3 "http://www.vishay.com/docs/31509/csc.pdf" H 6680 6645 50  0001 C CNN
+F 4 "Bussed" H 6680 6645 50  0001 C CNN "Notes"
 	1    6680 6645
 	1    0    0    -1
@@
 F 2 "Resistor_THT:R_Array_SIP6" V 7050 9495 50  0001 C CNN
 F 3 "http://www.vishay.com/docs/31509/csc.pdf" H 6675 9495 50  0001 C CNN
+F 4 "Bussed" H 6675 9495 50  0001 C CNN "Notes"
 	1    6675 9495
 	1    0    0    -1
@@
 F 2 "Resistor_THT:R_Array_SIP6" V 10275 1240 50  0001 C CNN
 F 3 "http://www.vishay.com/docs/31509/csc.pdf" H 9900 1240 50  0001 C CNN
+F 4 "Bussed" H 9900 1240 50  0001 C CNN "Notes"
 	1    9900 1240
 	1    0    0    -1
@@
 F 2 "Resistor_THT:R_Array_SIP6" V 10275 3880 50  0001 C CNN
 F 3 "http://www.vishay.com/docs/31509/csc.pdf" H 9900 3880 50  0001 C CNN
+F 4 "Bussed" H 9900 3880 50  0001 C CNN "Notes"
 	1    9900 3880
 	1    0    0    -1
@@
 F 2 "Resistor_THT:R_Array_SIP6" V 10270 9495 50  0001 C CNN
 F 3 "http://www.vishay.com/docs/31509/csc.pdf" H 9895 9495 50  0001 C CNN
+F 4 "Bussed" H 9895 9495 50  0001 C CNN "Notes"
 	1    9895 9495
 	1    0    0    -1
@@
 F 2 "Resistor_THT:R_Array_SIP6" V 7055 1240 50  0001 C CNN
 F 3 "http://www.vishay.com/docs/31509/csc.pdf" H 6680 1240 50  0001 C CNN
+F 4 "Bussed" H 6680 1240 50  0001 C CNN "Notes"
 	1    6680 1240
 	1    0    0    -1
@@
 F 2 "Resistor_THT:R_Array_SIP6" V 10275 6645 50  0001 C CNN
 F 3 "http://www.vishay.com/docs/31509/csc.pdf" H 9900 6645 50  0001 C CNN
+F 4 "Bussed" H 9900 6645 50  0001 C CNN "Notes"
 	1    9900 6645
 	1    0    0    -1
@@
 F 2 "Resistor_THT:R_Array_SIP10" V 2560 2725 50  0001 C CNN
 F 3 "http://www.vishay.com/docs/31509/csc.pdf" H 2640 2725 50  0001 C CNN
+F 4 "Independent" H 2640 2725 50  0001 C CNN "Notes"
 	2    2640 2725
 	0    1    1    0
@@
 F 2 "Resistor_THT:R_Array_SIP10" V 2560 2625 50  0001 C CNN
 F 3 "http://www.vishay.com/docs/31509/csc.pdf" H 2640 2625 50  0001 C CNN
+F 4 "Independent" H 2640 2625 50  0001 C CNN "Notes"
 	3    2640 2625
 	0    1    1    0
@@
 F 2 "Resistor_THT:R_Array_SIP10" V 2560 2525 50  0001 C CNN
 F 3 "http://www.vishay.com/docs/31509/csc.pdf" H 2640 2525 50  0001 C CNN
+F 4 "Independent" H 2640 2525 50  0001 C CNN "Notes"
 	4    2640 2525
 	0    1    1    0
@@
 F 2 "Resistor_THT:R_Array_SIP10" V 2560 2925 50  0001 C CNN
 F 3 "http://www.vishay.com/docs/31509/csc.pdf" H 2640 2925 50  0001 C CNN
+F 4 "Independent" H 2640 2925 50  0001 C CNN "Notes"
 	5    2640 2925
 	0    1    1    0
@@
 Wire Wire Line
 	2790 2625 3315 2625
+$Comp
+L Device:R_Pack05_SIP_Split RN9
+U 1 1 63C134E3
+P 2640 3125
+F 0 "RN9" V 2600 3375 50  0000 C CNN
+F 1 "100" V 2600 2930 50  0000 C CNN
+F 2 "Resistor_THT:R_Array_SIP10" V 2560 3125 50  0001 C CNN
+F 3 "http://www.vishay.com/docs/31509/csc.pdf" H 2640 3125 50  0001 C CNN
+F 4 "Independent" H 2640 3125 50  0001 C CNN "Notes"
+	1    2640 3125
+	0    1    1    0
+$EndComp
 Wire Bus Line
 	13345 2405 13345 2805
@@
 Wire Bus Line
 	3415 2625 3415 4050
-$Comp
-L Device:R_Pack05_SIP_Split RN9
-U 1 1 63C134E3
-P 2640 3125
-F 0 "RN9" V 2600 3375 50  0000 C CNN
-F 1 "100" V 2600 2930 50  0000 C CNN
-F 2 "Resistor_THT:R_Array_SIP10" V 2560 3125 50  0001 C CNN
-F 3 "http://www.vishay.com/docs/31509/csc.pdf" H 2640 3125 50  0001 C CNN
-	1    2640 3125
-	0    1    1    0
-$EndComp
 $EndSCHEMATC
